File: hardware/picomax/picomax.kicad_sch (KiCad schematic)
At the start: 4 parts, among them U2 MAX4619CPE+, U3 SC0915, U4 PIC16LF1936-I/SS

Commit message: Updated schematics
Connections:
- net TRIG_IN_PIN: now also U4.2 (VCAP/~SS/SEG12/SRNQ/C2OUT/C12IN0-/AN0/RA0)
- net I2C_SCL_PIN: now reaches U4.14 (SEG6/SCL/SCK/RC3)
- net I2C_SCL_PIN: now also U3.22 (GP17)
- net I2C_SDA_PIN: now reaches U4.15 (RC4/SDI/SDA/T1G/SEG11)
- net I2C_SDA_PIN: now also U3.21 (GP16)
- net PIC_START_READ_PIN: now reaches U3.9 (GP6)
- net PIC_GLITCH_FAIL_PIN: no longer names the net of U3.11 (GP8)
- net PIC_GLITCH_FAIL_PIN: no longer U4.3 (SEG7/C12IN1-/AN1/RA1)
- net PIC_GLITCH_SUCC_PIN: no longer names the net of U4.4 (COM2/DACOUT/C2IN+/VREF-/AN2/RA2)
- net PIC_GLITCH_SUCC_PIN: no longer U3.12 (GP9)
- net PIC_OUT_PIN: no longer names the net of U3.10 (GP7)
- net PIC_OUT_PIN: no longer U4.2 (VCAP/~SS/SEG12/SRNQ/C2OUT/C12IN0-/AN0/RA0)
- new net START_READ_PIN: U4.3 (SEG7/C12IN1-/AN1/RA1)
Changed lines of the file:
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@@
     (effects (font (size 1.27 1.27)) (justify left top))
   )
-  (text_box "TRIG_IN_PIN starts the glitching process and must be connected to some source.\nWhich soure depends on what you want to use as a reference to glitch\n\nI have it connected to nMCLR from the Pico to start glitching after the programming mode is enabled"
+  (text_box "TRIG_IN_PIN starts the glitching process and must be connected to some source.\nWhich source depends on what you want to use as a reference to glitch\n\nI have it connected to nMCLR from the Pico to start glitching after the programming mode is enabled"
     (at 17.78 127 0) (size 48.26 17.78)
     (stroke (width 0) (type default))
@@
     )
   )
+  (global_label "I2C_SCL_PIN" (shape input) (at 43.18 82.55 180) (fields_autoplaced)
+    (effects (font (size 1.27 1.27)) (justify right))
+    (property "Intersheetrefs" "${INTERSHEET_REFS}" (at 28.5418 82.55 0)
+      (effects (font (size 1.27 1.27)) (justify right) hide)
+    )
+  )
   (global_label "Vdd" (shape input) (at 127 166.37 180) (fields_autoplaced)
     (effects (font (size 1.27 1.27)) (justify right))
@@
     )
   )
-  (global_label "PIC_GLITCH_SUCC_PIN" (shape input) (at 43.18 29.21 180) (fields_autoplaced)
+  (global_label "I2C_SDA_PIN" (shape input) (at 43.18 69.85 180) (fields_autoplaced)
     (effects (font (size 1.27 1.27)) (justify right))
-    (property "Intersheetrefs" "${INTERSHEET_REFS}" (at 19.4703 29.21 0)
+    (property "Intersheetrefs" "${INTERSHEET_REFS}" (at 28.4813 69.85 0)
       (effects (font (size 1.27 1.27)) (justify right) hide)
     )
@@
     (effects (font (size 1.27 1.27)) (justify right))
     (property "Intersheetrefs" "${INTERSHEET_REFS}" (at 120.7076 143.51 0)
-      (effects (font (size 1.27 1.27)) (justify right) hide)
-    )
-  )
-  (global_label "PIC_OUT_PIN" (shape input) (at 39.37 195.58 180) (fields_autoplaced)
-    (effects (font (size 1.27 1.27)) (justify right))
-    (property "Intersheetrefs" "${INTERSHEET_REFS}" (at 24.5503 195.58 0)
-      (effects (font (size 1.27 1.27)) (justify right) hide)
-    )
-  )
-  (global_label "PIC_OUT_PIN" (shape input) (at 43.18 46.99 180) (fields_autoplaced)
-    (effects (font (size 1.27 1.27)) (justify right))
-    (property "Intersheetrefs" "${INTERSHEET_REFS}" (at 28.3603 46.99 0)
       (effects (font (size 1.27 1.27)) (justify right) hide)
     )
@@
     )
   )
+  (global_label "PIC_START_READ_PIN" (shape input) (at 39.37 193.04 180) (fields_autoplaced)
+    (effects (font (size 1.27 1.27)) (justify right))
+    (property "Intersheetrefs" "${INTERSHEET_REFS}" (at 16.9304 193.04 0)
+      (effects (font (size 1.27 1.27)) (justify right) hide)
+    )
+  )
   (global_label "nMCLR" (shape input) (at 90.17 195.58 0) (fields_autoplaced)
     (effects (font (size 1.27 1.27)) (justify left))
     (property "Intersheetrefs" "${INTERSHEET_REFS}" (at 99.2443 195.58 0)
+      (effects (font (size 1.27 1.27)) (justify left) hide)
+    )
+  )
+  (global_label "I2C_SDA_PIN" (shape input) (at 90.17 185.42 0) (fields_autoplaced)
+    (effects (font (size 1.27 1.27)) (justify left))
+    (property "Intersheetrefs" "${INTERSHEET_REFS}" (at 104.8687 185.42 0)
       (effects (font (size 1.27 1.27)) (justify left) hide)
     )
@@
     )
   )
-  (global_label "PIC_GLITCH_FAIL_PIN" (shape input) (at 43.18 41.91 180) (fields_autoplaced)
+  (global_label "TRIG_IN_PIN" (shape input) (at 43.18 46.99 180) (fields_autoplaced)
     (effects (font (size 1.27 1.27)) (justify right))
-    (property "Intersheetrefs" "${INTERSHEET_REFS}" (at 20.7402 41.91 0)
+    (property "Intersheetrefs" "${INTERSHEET_REFS}" (at 29.086 46.99 0)
+      (effects (font (size 1.27 1.27)) (justify right) hide)
+    )
+  )
+  (global_label "START_READ_PIN" (shape input) (at 43.18 41.91 180) (fields_autoplaced)
+    (effects (font (size 1.27 1.27)) (justify right))
+    (property "Intersheetrefs" "${INTERSHEET_REFS}" (at 24.8528 41.91 0)
       (effects (font (size 1.27 1.27)) (justify right) hide)
     )
@@
     (property "Intersheetrefs" "${INTERSHEET_REFS}" (at 185.8463 36.83 0)
       (effects (font (size 1.27 1.27)) (justify left) hide)
-    )
-  )
-  (global_label "PIC_GLITCH_FAIL_PIN" (shape input) (at 39.37 198.12 180) (fields_autoplaced)
-    (effects (font (size 1.27 1.27)) (justify right))
-    (property "Intersheetrefs" "${INTERSHEET_REFS}" (at 16.9302 198.12 0)
-      (effects (font (size 1.27 1.27)) (justify right) hide)
     )
   )
@@
     )
   )
-  (global_label "PIC_GLITCH_SUCC_PIN" (shape input) (at 39.37 200.66 180) (fields_autoplaced)
-    (effects (font (size 1.27 1.27)) (justify right))
-    (property "Intersheetrefs" "${INTERSHEET_REFS}" (at 15.6603 200.66 0)
-      (effects (font (size 1.27 1.27)) (justify right) hide)
-    )
-  )
   (global_label "nMCLR" (shape input) (at 43.18 95.25 180) (fields_autoplaced)
     (effects (font (size 1.27 1.27)) (justify right))
@@
     )
   )
+  (global_label "I2C_SCL_PIN" (shape input) (at 90.17 187.96 0) (fields_autoplaced)
+    (effects (font (size 1.27 1.27)) (justify left))
+    (property "Intersheetrefs" "${INTERSHEET_REFS}" (at 104.8082 187.96 0)
+      (effects (font (size 1.27 1.27)) (justify left) hide)
+    )
+  )
